File: Anteres-Receiver.kicad_pcb (KiCad board)
At the start: 2 copper layers, 40 x 40 mm, 55 parts, among them J301 PS2 Male Socket, J501 Debugger Pin, SW201 SW_SPST, U201 STM32G070KBTx, U401 CC1101RGPR, Y401 27MHz

Commit message: :minidisc: fixed dvdd of cc1101 pin unconnected
Connections:
- U401 pad 4: unconnected-(U401-DVDD-Pad4) -> +3V3
Routing:
- net +3V3: track 131.4 -> 133.7 mm, vias 8 -> 9
Other:
- board text added: "Project Antares - Recv v1.0.1 ${CURRENT_DATE}"
- board text removed: "Project Antares - Recv v1.0.0 ${CURRENT_DATE}"
