File: Anteres-Receiver.kicad_sch (KiCad schematic)
At the start: 0 parts

Commit message: :memo: updated schemati and pcb information
Other:
- company: Ouroboros Embedded Education -> Ouroboros Embedded Development
- title: Project Antares - Receiver -> Project Antares - Receiver Schematic
Changed lines of the file:
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@@
 	(paper "A4")
 	(title_block
-		(title "Project Antares - Receiver")
-		(date "2024-08-22")
-		(rev "Rev 1")
-		(company "Ouroboros Embedded Education")
+		(title "Project Antares - Receiver Schematic")
+		(date "2024-08-23")
+		(rev "1.0.0")
+		(company "Ouroboros Embedded Development")
 		(comment 1 "Pablo Jean Rozario")
 	)
