File: debugging.kicad_sch (KiCad schematic)
At the start: 6 parts, among them J501 Debugger Pin

Commit message: :memo: updated schemati and pcb information
Other:
- company: Ouroboros Embedded Education -> Ouroboros Embedded Development
- title: Project Antares - Receiver -> Project Antares - Receiver Schematic
Changed lines of the file:
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@@
 	(paper "A4")
 	(title_block
-		(title "Project Antares - Receiver")
-		(date "2024-08-22")
-		(rev "Rev 1")
-		(company "Ouroboros Embedded Education")
+		(title "Project Antares - Receiver Schematic")
+		(date "2024-08-23")
+		(rev "1.0.0")
+		(company "Ouroboros Embedded Development")
 		(comment 1 "Pablo Jean Rozario")
 	)

Commit message: :minidisc: fixed dvdd of cc1101 pin unconnected
Parts:
- R501, R502, R503, R504, R505: LCSC C25202 -> C22859; PN 0603WAJ0100T5E -> 0603WAF100JT5E
Changed lines of the file:
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@@
 	(title_block
 		(title "Project Antares - Receiver Schematic")
-		(date "2024-08-23")
-		(rev "1.0.0")
+		(date "2024-08-24")
+		(rev "1.0.1")
 		(company "Ouroboros Embedded Development")
 		(comment 1 "Pablo Jean Rozario")
@@
 			)
 		)
-		(property "LCSC" "C25202"
+		(property "LCSC" "C22859"
 			(at 130.81 90.17 0)
 			(effects
@@
 			)
 		)
-		(property "PN" "0603WAJ0100T5E"
+		(property "PN" "0603WAF100JT5E"
 			(at 130.81 90.17 0)
 			(effects
@@
 			)
 		)
-		(property "LCSC" "C25202"
+		(property "LCSC" "C22859"
 			(at 130.81 97.79 0)
 			(effects
@@
 			)
 		)
-		(property "PN" "0603WAJ0100T5E"
+		(property "PN" "0603WAF100JT5E"
 			(at 130.81 97.79 0)
 			(effects
@@
 			)
 		)
-		(property "LCSC" "C25202"
+		(property "LCSC" "C22859"
 			(at 130.81 95.25 0)
 			(effects
@@
 			)
 		)
-		(property "PN" "0603WAJ0100T5E"
+		(property "PN" "0603WAF100JT5E"
 			(at 130.81 95.25 0)
 			(effects
@@
 			)
 		)
-		(property "LCSC" "C25202"
+		(property "LCSC" "C22859"
 			(at 130.81 100.33 0)
 			(effects
@@
 			)
 		)
-		(property "PN" "0603WAJ0100T5E"
+		(property "PN" "0603WAF100JT5E"
 			(at 130.81 100.33 0)
 			(effects
@@
 			)
 		)
-		(property "LCSC" "C25202"
+		(property "LCSC" "C22859"
 			(at 130.81 92.71 0)
 			(effects
@@
 			)
 		)
-		(property "PN" "0603WAJ0100T5E"
+		(property "PN" "0603WAF100JT5E"
 			(at 130.81 92.71 0)
 			(effects
