File: mcu.kicad_sch (KiCad schematic)
At the start: 15 parts, among them SW201 SW_SPST, U201 STM32G070KBTx

Commit message: :memo: updated schemati and pcb information
Other:
- company: Ouroboros Embedded Education -> Ouroboros Embedded Development
- title: Project Antares - Receiver -> Project Antares - Receiver Schematic
Changed lines of the file:
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@@
 	(paper "A4")
 	(title_block
-		(title "Project Antares - Receiver")
-		(date "2024-08-22")
-		(rev "Rev 1")
-		(company "Ouroboros Embedded Education")
+		(title "Project Antares - Receiver Schematic")
+		(date "2024-08-23")
+		(rev "1.0.0")
+		(company "Ouroboros Embedded Development")
 		(comment 1 "Pablo Jean Rozario")
 	)

Commit message: :minidisc: fixed dvdd of cc1101 pin unconnected
Parts:
- R201, R202, R206: LCSC C2930027 -> C25804; PN FRC0603J103TS -> 0603WAF1002T5E
- R203: LCSC C2907127 -> C23345; PN FRC0603J221 TS -> 0603WAF220JT5E
- R204, R205: LCSC C25201 -> C22775; PN 0603WAJ0101T5E -> 0603WAF1000T5E
Changed lines of the file:
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@@
 	(title_block
 		(title "Project Antares - Receiver Schematic")
-		(date "2024-08-23")
-		(rev "1.0.0")
+		(date "2024-08-24")
+		(rev "1.0.1")
 		(company "Ouroboros Embedded Development")
 		(comment 1 "Pablo Jean Rozario")
@@
 			)
 		)
-		(property "LCSC" "C25201"
+		(property "LCSC" "C22775"
 			(at 224.79 99.06 0)
 			(effects
@@
 			)
 		)
-		(property "PN" "0603WAJ0101T5E"
+		(property "PN" "0603WAF1000T5E"
 			(at 224.79 99.06 0)
 			(effects
@@
 			)
 		)
-		(property "LCSC" "C25201"
+		(property "LCSC" "C22775"
 			(at 224.79 104.14 0)
 			(effects
@@
 			)
 		)
-		(property "PN" "0603WAJ0101T5E"
+		(property "PN" "0603WAF1000T5E"
 			(at 224.79 104.14 0)
 			(effects
@@
 			)
 		)
-		(property "LCSC" "C2930027"
+		(property "LCSC" "C25804"
 			(at 105.41 119.38 0)
 			(effects
@@
 			)
 		)
-		(property "PN" "FRC0603J103TS"
+		(property "PN" "0603WAF1002T5E"
 			(at 105.41 119.38 0)
 			(effects
@@
 			)
 		)
-		(property "LCSC" "C2930027"
+		(property "LCSC" "C25804"
 			(at 224.79 41.91 0)
 			(effects
@@
 			)
 		)
-		(property "PN" "FRC0603J103TS"
+		(property "PN" "0603WAF1002T5E"
 			(at 224.79 41.91 0)
 			(effects
@@
 			)
 		)
-		(property "LCSC" "C2907127"
+		(property "LCSC" "C23345"
 			(at 224.79 93.98 0)
 			(effects
@@
 			)
 		)
-		(property "PN" "FRC0603J221 TS"
+		(property "PN" "0603WAF220JT5E"
 			(at 224.79 93.98 0)
 			(effects
@@
 			)
 		)
-		(property "LCSC" "C2930027"
+		(property "LCSC" "C25804"
 			(at 234.95 33.02 0)
 			(effects
@@
 			)
 		)
-		(property "PN" "FRC0603J103TS"
+		(property "PN" "0603WAF1002T5E"
 			(at 234.95 33.02 0)
 			(effects
