File: ps2_conn.kicad_sch (KiCad schematic)
At the start: 9 parts, among them J301 PS2 Male Socket

Commit message: :memo: updated schemati and pcb information
Other:
- company: Ouroboros Embedded Education -> Ouroboros Embedded Development
- title: Project Antares - Receiver -> Project Antares - Receiver Schematic
Changed lines of the file:
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@@
 	(paper "A4")
 	(title_block
-		(title "Project Antares - Receiver")
-		(date "2024-08-22")
-		(rev "Rev 1")
-		(company "Ouroboros Embedded Education")
+		(title "Project Antares - Receiver Schematic")
+		(date "2024-08-23")
+		(rev "1.0.0")
+		(company "Ouroboros Embedded Development")
 		(comment 1 "Pablo Jean Rozario")
 	)

Commit message: :minidisc: fixed dvdd of cc1101 pin unconnected
Parts:
- R301, R302: LCSC C25999 -> C23162; PN 0603WAJ0472T5E -> 0603WAF4701T5E
Changed lines of the file:
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@@
 	(title_block
 		(title "Project Antares - Receiver Schematic")
-		(date "2024-08-23")
-		(rev "1.0.0")
+		(date "2024-08-24")
+		(rev "1.0.1")
 		(company "Ouroboros Embedded Development")
 		(comment 1 "Pablo Jean Rozario")
@@
 			)
 		)
-		(property "LCSC" "C25999"
+		(property "LCSC" "C23162"
 			(at 113.03 71.12 0)
 			(effects
@@
 			)
 		)
-		(property "PN" "0603WAJ0472T5E"
+		(property "PN" "0603WAF4701T5E"
 			(at 113.03 71.12 0)
 			(effects
@@
 			)
 		)
-		(property "LCSC" "C25999"
+		(property "LCSC" "C23162"
 			(at 120.65 71.12 0)
 			(effects
@@
 			)
 		)
-		(property "PN" "0603WAJ0472T5E"
+		(property "PN" "0603WAF4701T5E"
 			(at 120.65 71.12 0)
 			(effects
